File: hardware/cybermix.kicad_pcb (KiCad board)
At the start: 4 copper layers, 205 x 123 mm, 31 parts, among them J1 PINHD_1x16_Male, J2 PINHD_1x4_Male, SW1 SW_Push, SW2 SW_Push, U1 XIAO-RP2040-DIP, U2 2717

Commit message: update files
Parts:
- moved D4 1.12 mm to (158.0, 150.0), turned to -90 degrees
- moved D6 1.12 mm to (186.2, 150.0), turned to -90 degrees
- moved D1 1.00 mm to (96.0, 150.0), turned to -90 degrees
- moved D2 1.00 mm to (130.0, 150.0), turned to -90 degrees
- moved D3 1.00 mm to (144.0, 150.0), turned to 90 degrees
- moved D5 1.00 mm to (172.0, 150.0), turned to 90 degrees
- moved D7 1.00 mm to (200.0, 150.0), turned to 90 degrees
- moved D8 1.00 mm to (214.0, 150.0), turned to -90 degrees
- moved D9 1.00 mm to (228.0, 150.0), turned to 90 degrees
Routing:
- net Net-(ADC1-GND): track 721.4 -> 883.3 mm, vias 10 -> 12
- net Net-(ADC1-VCC): track 687.3 -> 767.6 mm, vias 10 -> 14
- net Net-(D10-DIN): track 118.0 -> 149.4 mm
- net Net-(D1-DOUT): track 39.8 -> 35.4 mm
- net Net-(D5-DOUT): track 19.4 -> 16.9 mm
- net Net-(D8-DOUT): track 18.8 -> 16.6 mm
- net Net-(D7-DOUT): track 18.8 -> 16.7 mm
- net Net-(D6-DOUT): track 18.6 -> 16.8 mm
- net Net-(U1-GPIO26/ADC0/A0): track 76.5 -> 78.2 mm
- net Net-(D4-DOUT): track 18.9 -> 17.3 mm
- net Net-(D3-DOUT): track 18.8 -> 17.3 mm
- net Net-(D2-DOUT): track 18.2 -> 16.9 mm
Other:
- copper layers 4 -> 2
